File: PCB_project/hpm_dap.kicad_pcb (KiCad board)
At the start: 2 copper layers, 28 x 17 mm, 45 parts, among them J1 USB_C_Receptacle_USB2.0_16P, J2 302-S101, SW1 SW_Push, U1 HPM5301IEGx, U2 TPS82130, X1 24MHz

Commit message: PCB layout 完毕
Parts:
- removed C2: 0.1uF, Capacitor_SMD:C_0402_1005Metric
- added D4: LED, LED_SMD:LED_0603_1608Metric, F.Cu at (65.4, 36.3)
- added D5: LED, LED_SMD:LED_0603_1608Metric, F.Cu at (65.4, 37.9)
- added R10: 33Ω, Resistor_SMD:R_0402_1005Metric, B.Cu at (77.2, 39.1)
- added R11: 33Ω, Resistor_SMD:R_0402_1005Metric, B.Cu at (78.2, 39.1)
- added R8: 1kΩ, Resistor_SMD:R_0402_1005Metric, F.Cu at (68.3, 38.2)
- added R9: 1kΩ, Resistor_SMD:R_0402_1005Metric, F.Cu at (67.9, 36.5)
- C10, C11, C13, C14, C18, C4, C5, C6, C8, C9: moved to B.Cu
- RN2: moved to F.Cu
- moved C15 40.2 mm to (79.0, 33.4), turned to 180 degrees
- moved C16 40.1 mm to (79.0, 34.3), turned to 180 degrees
- moved C5 39.2 mm to (75.1, 29.9), turned to 90 degrees
- moved C11 38.9 mm to (75.8, 36.7), turned to 90 degrees
- moved C8 38.7 mm to (73.1, 36.7), turned to 90 degrees
- moved C10 38.7 mm to (74.9, 36.7), turned to 90 degrees
- moved C9 38.7 mm to (74.0, 36.7), turned to 90 degrees
- moved C17 38.3 mm to (76.3, 39.1), turned to -90 degrees
- moved C13 37.8 mm to (76.3, 34.4), turned to 180 degrees
- moved C18 37.5 mm to (76.3, 39.1), turned to -90 degrees
- moved C6 37.2 mm to (73.3, 29.9), turned to 90 degrees
- moved C14 37.0 mm to (76.3, 35.3), turned to 180 degrees
- moved R5 11.9 mm to (62.6, 30.4), turned to -90 degrees
- moved D3 11.4 mm to (78.2, 30.6), turned to 0 degrees
- moved SW1 5.09 mm to (65.2, 32.8), turned to -90 degrees
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Connections:
- D2 pad 1: unconnected-(D2-Pad1) -> /SWDIO/JTAG_TMS
- D2 pad 3: unconnected-(D2-Pad3) -> /SWCLK/JTAG_TCK
- D2 pad 6: unconnected-(D2-Pad6) -> /SWRST/JTAG_TRST
- D3 pad 1: unconnected-(D3-Pad1) -> /uart_rx
- D3 pad 3: unconnected-(D3-Pad3) -> /uart_tx
- D3 pad 4: unconnected-(D3-Pad4) -> /JTAG_TDI
- D3 pad 6: unconnected-(D3-Pad6) -> /JTAG_TDO
- RN1 pad 1: Net-(RN1-R1.1) -> unconnected-(RN1-R1.1-Pad1)
- RN1 pad 8: /core/SPI_CS -> unconnected-(RN1-R1.2-Pad8)
- RN2 pad 1: Net-(RN2-R1.1) -> unconnected-(RN2-R1.1-Pad1)
- RN2 pad 5: /core/SPI_CS -> /JTAG_TDI
- RN2 pad 6: /SWCLK/JTAG_TCK -> /JTAG_TDO
- RN2 pad 7: /JTAG_TDO -> /SWCLK/JTAG_TCK
- RN2 pad 8: /JTAG_TDI -> unconnected-(RN2-R1.2-Pad8)
- U1 pad 11: /uart_rx -> Net-(U1D-PA01/TMR1.CAPT0/URT0.RXD/TRGM0.P01/ACMP.COMP0)
- U1 pad 12: /uart_tx -> Net-(U1D-PA00/TMR1.COMP0/URT0.TXD/TRGM0.P00)
- U1 pad 22: Net-(RN2-R1.1) -> Net-(RN2-R4.1)
- U1 pad 23: Net-(RN2-R2.1) -> Net-(RN2-R3.1)
- U1 pad 24: Net-(RN2-R3.1) -> Net-(RN2-R2.1)
- U1 pad 25: Net-(RN2-R4.1) -> /core/SPI_CS
- U1 pad 42: Net-(RN1-R1.1) -> /core/SPI_CS
- U1 pad 48: unconnected-(U1D-PA05/TMR1.COMP2/URT1.DE/URT1.RTS/SPI0.SCLK/TRGM0.P05/JTAG.TDI-Pad48) -> /core/LED
Routing:
- net +3.3V: track 0.00 -> 63.6 mm, vias 0 -> 7
- net /SWCLK/JTAG_TCK: track 0.00 -> 19.1 mm, vias 0 -> 2
- net /uart_rx: track 0.00 -> 19.1 mm
- net /uart_tx: track 0.00 -> 19.1 mm
- net /JTAG_TDI: track 0.00 -> 17.6 mm, vias 0 -> 2
- net /core/USB_D-: track 0.00 -> 15.7 mm, vias 0 -> 1
- net Net-(F1-Pad1): track 0.00 -> 15.5 mm
- net /core/USB_D+: track 0.00 -> 15.4 mm, vias 0 -> 1
- net /JTAG_TDO: track 0.00 -> 11.9 mm, vias 0 -> 2
- net VBUS: track 0.00 -> 11.0 mm, vias 0 -> 1
- net /core/SPI_CS: track 0.00 -> 10.6 mm, vias 0 -> 2
- net /SWDIO/JTAG_TMS: track 0.00 -> 9.33 mm, vias 0 -> 1
- net /SWRST/JTAG_TRST: track 0.00 -> 8.55 mm, vias 0 -> 2
- net /core/BOOT1: track 9.26 -> 14.2 mm
- net GND: track 0.00 -> 4.63 mm, vias 0 -> 46
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- added copper zone on F.Cu, net +3.3V
- added copper zone on B.Cu, net GND
- added copper zone on F.Cu, net GND
- added copper zone on F.Cu, net VBUS
Other:
- outline, holes or cut-outs redrawn
- board text added: "BOOT"
- board text added: "C"
- board text added: "D"
- board text added: "G"
- board text added: "NC"
- board text added: "R"
- board text added: "RX"
- board text added: "TDI"
- board text added: "TDO"
- board text added: "TX"
