File: PCB_project/hpm_dap.kicad_sch (KiCad schematic)
At the start: 8 parts, among them J1 USB_C_Receptacle_USB2.0_16P, J2 302-S101

Commit message: PCB layout 完毕
Parts:
- added D4, D5: LED, LED_SMD:LED_0603_1608Metric, symbol Device:LED
- added R8, R9: 1kΩ, Resistor_SMD:R_0402_1005Metric, symbol Device:R
Connections:
- net +3.3V: now also R9.1
- net GND: now also D4.1 (K), D5.1 (K)
- net JTAG_TDI: now also D3.4
- net JTAG_TDO: now also D3.6
- net SWCLK/JTAG_TCK: now also D2.3
- net SWDIO/JTAG_TMS: now also D2.1
- net SWRST/JTAG_TRST: now also D2.6
- net uart_rx: now also D3.1
- net uart_tx: now also D3.3
- new net: D5.2 (A), R8.1
- new net: D4.2 (A), R9.2
- new net core/LED: R8.2
Other:
- sheet core ports: added LED; removed none
- moved on the sheet: D3
